File: pcb/Schematic.brd (EAGLE design)
At the start: 40.3 x 53.3 mm, 5 parts

Commit message: board layout changes
Parts:
- turned SL2 to 180 degrees
Routing:
- net LOAD+: track 17.8 -> 19.6 mm
- net 3V3: track 32.3 -> 33.1 mm
- net SWITCH: track 9.94 -> 9.41 mm
Changed lines of the file:
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@@
 <param name="RoutingGrid" value="50mil"/>
 <param name="AutoGrid" value="1"/>
-<param name="Efforts" value="0"/>
+<param name="Efforts" value="2"/>
 <param name="TopRouterVariant" value="1"/>
 <param name="tpViaShape" value="round"/>
@@
 <attribute name="OC_NEWARK" value="unknown" x="59.69" y="26.67" size="1.778" layer="27" rot="R90" display="off"/>
 </element>
-<element name="SL2" library="con-amp-quick" library_urn="urn:adsk.eagle:library:125" package="02P" value="" x="59.69" y="66.04" rot="R270">
-<attribute name="MF" value="" x="59.69" y="66.04" size="1.778" layer="27" rot="R270" display="off"/>
-<attribute name="MPN" value="" x="59.69" y="66.04" size="1.778" layer="27" rot="R270" display="off"/>
-<attribute name="OC_FARNELL" value="unknown" x="59.69" y="66.04" size="1.778" layer="27" rot="R270" display="off"/>
-<attribute name="OC_NEWARK" value="unknown" x="59.69" y="66.04" size="1.778" layer="27" rot="R270" display="off"/>
+<element name="SL2" library="con-amp-quick" library_urn="urn:adsk.eagle:library:125" package="02P" value="" x="59.69" y="66.04" rot="R180">
+<attribute name="MF" value="" x="59.69" y="66.04" size="1.778" layer="27" rot="R180" display="off"/>
+<attribute name="MPN" value="" x="59.69" y="66.04" size="1.778" layer="27" rot="R180" display="off"/>
+<attribute name="OC_FARNELL" value="unknown" x="59.69" y="66.04" size="1.778" layer="27" rot="R180" display="off"/>
+<attribute name="OC_NEWARK" value="unknown" x="59.69" y="66.04" size="1.778" layer="27" rot="R180" display="off"/>
 </element>
 </elements>
@@
 <contactref element="PWR1" pad="P1"/>
 <contactref element="SL1" pad="1"/>
-<wire x1="53.34" y1="19.05" x2="59.69" y2="25.4" width="0.1524" layer="16"/>
+<wire x1="53.34" y1="19.05" x2="59.69" y2="25.4" width="0.3048" layer="16"/>
 </signal>
 <signal name="L">
 <contactref element="SL1" pad="2"/>
 <contactref element="PWR1" pad="P2"/>
-<wire x1="53.34" y1="34.29" x2="59.69" y2="27.94" width="0.1524" layer="16"/>
+<wire x1="53.34" y1="34.29" x2="59.69" y2="27.94" width="0.3048" layer="16"/>
 </signal>
 <signal name="3V3">
 <contactref element="PWR1" pad="P4"/>
 <contactref element="CORE" pad="24"/>
-<wire x1="26.67" y1="42.3672" x2="26.67" y2="58.42" width="0.1524" layer="16"/>
-<wire x1="25.4508" y1="41.148" x2="26.67" y2="42.3672" width="0.1524" layer="16"/>
-<wire x1="25.4508" y1="26.67" x2="25.4508" y2="41.148" width="0.1524" layer="16"/>
-<wire x1="25.4508" y1="26.67" x2="25.4" y2="26.67" width="0.1524" layer="16"/>
+<wire x1="24.13" y1="55.0672" x2="26.67" y2="58.42" width="0.1524" layer="16"/>
+<wire x1="24.1808" y1="42.418" x2="24.13" y2="55.0672" width="0.1524" layer="16"/>
+<wire x1="24.1808" y1="27.94" x2="24.1808" y2="42.418" width="0.1524" layer="16"/>
+<wire x1="24.1808" y1="27.94" x2="25.4" y2="26.67" width="0.1524" layer="16"/>
 </signal>
 <signal name="GND">
@@
 <wire x1="59.5884" y1="67.3608" x2="41.91" y2="67.3608" width="0.1524" layer="1"/>
 <wire x1="41.91" y1="67.3608" x2="41.91" y2="67.31" width="0.1524" layer="1"/>
-<wire x1="59.5884" y1="67.3608" x2="59.69" y2="67.31" width="0.1524" layer="1"/>
+<wire x1="59.5884" y1="67.3608" x2="60.96" y2="66.04" width="0.1524" layer="1"/>
 </signal>
 <signal name="LOAD-">
 <contactref element="SL2" pad="2"/>
 <contactref element="RELAY1" pad="1"/>
-<wire x1="32.9184" y1="62.3316" x2="31.8516" y2="62.3316" width="0.1524" layer="16"/>
-<wire x1="35.3568" y1="64.77" x2="32.9184" y2="62.3316" width="0.1524" layer="16"/>
-<wire x1="59.69" y1="64.77" x2="35.3568" y2="64.77" width="0.1524" layer="16"/>
+<wire x1="31.9024" y1="64.3636" x2="31.8516" y2="62.3316" width="0.1524" layer="16"/>
+<wire x1="34.0868" y1="66.04" x2="31.9024" y2="64.3636" width="0.1524" layer="16"/>
+<wire x1="58.42" y1="66.04" x2="34.0868" y2="66.04" width="0.1524" layer="16"/>
 <wire x1="31.8516" y1="62.3316" x2="31.75" y2="62.23" width="0.1524" layer="16"/>
 </signal>
@@
 <contactref element="CORE" pad="20"/>
 <contactref element="RELAY1" pad="2"/>
-<wire x1="34.29" y1="63.7032" x2="34.29" y2="67.31" width="0.1524" layer="1"/>
-<wire x1="36.7284" y1="61.2648" x2="34.29" y2="63.7032" width="0.1524" layer="1"/>
+<wire x1="35.433" y1="64.4652" x2="34.29" y2="67.31" width="0.1524" layer="1"/>
+<wire x1="36.7284" y1="61.2648" x2="35.433" y2="64.4652" width="0.1524" layer="1"/>
 <wire x1="36.7284" y1="58.5216" x2="36.7284" y2="61.2648" width="0.1524" layer="1"/>
 <wire x1="36.7284" y1="58.5216" x2="36.83" y2="58.42" width="0.1524" layer="1"/>
